File: gbsc-sync-combiner-v2/gbsc-sync-combiner-v2.kicad_pcb (KiCad board)
At the start: 2 copper layers, 33 x 47 mm, 13 parts, among them J1 DB15_Female_HighDensity_Mount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, J2 JST-XH, J3 JST-XH, U1 74LS86

Commit message: Adjust silks
Other:
- board text added: "25 x 39mm M3"
- board text added: "GBS-C Sync Combiner v1.0 c. 11/2021 github.com/Softdrink117/gbsc-sync-combiner CERN-OHL-W"

Commit message: Minor adjustments
Parts:
- added G***: LOGO, board_graphics:sft_logo, F.Cu at (107.5, 93.0)
- moved H2 1.00 mm to (101.0, 93.0)
- moved H3 1.00 mm to (126.0, 93.0)
- moved J2 0.50 mm to (110.0, 87.0)
- moved J3 0.50 mm to (110.0, 76.5)
- moved J1 0.46 mm to (104.1, 77.2)
Routing:
- net GND: track 124.5 -> 123.6 mm
- net /HSync: track 45.6 -> 46.5 mm
- net Net-(J1-Pad0): track 37.4 -> 38.2 mm
- net /VSync: track 45.3 -> 46.0 mm
Other:
- board size 33 x 47 mm -> 33 x 48 mm
- board text added: "GBS-C Sync Combiner v1.0 c. 11/2021 Details on Github: Softdrink117/gbsc-sync-combiner CERN-OHL-W"
- board text added: "Mounting: 25 x 40mm M3"
- board text removed: "25 x 39mm M3"
- board text removed: "GBS-C Sync Combiner v1.0 c. 11/2021 github.com/Softdrink117/gbsc-sync-combiner CERN-OHL-W"

Commit message: Minor tweaks
Other:
- board text added: "Power IN"
- board text added: "RGBHV IN"
- board text added: "RGBS OUT"
