File: gbsc-control-board/gbsc-control-board.kicad_sch (KiCad schematic)
At the start: 17 parts

Commit message: Layout and route control board
Parts:
- C1, C2: renamed from C?; footprint (none) -> Capacitor_THT:C_Disc_D3.0mm_W1.6mm_P2.50mm
- H1, H2, H3, H4: renamed from H?; footprint (none) -> MountingHole:MountingHole_3.2mm_M3_Pad; now left out of the parts list
- J1, J2, J3: renamed from J?; footprint (none) -> GBSC_Sync_Combiner_Footprints:Solder_Pad_2x4mm; now left out of the parts list
- J4: renamed from J?; footprint (none) -> TerminalBlock_MetzConnect:TerminalBlock_MetzConnect_Type059_RT06303HBWC_1x03_P3.50mm_Horizontal
- J5: renamed from J?; footprint (none) -> Connector_JST:JST_XH_B4B-XH-A_1x04_P2.50mm_Vertical
- SW1: renamed from SW?; value RotaryEncoder_Switch -> EC11 Rotary Encoder; footprint (none) -> Rotary_Encoder:RotaryEncoder_Alps_EC11E-Switch_Vertical_H20mm
- U2: renamed from U?; footprint (none) -> GBSC_Sync_Combiner_Footprints:SSD1306_OLED_0.96-Inch
- gave numbers to parts that had none: 4
Connections:
- net +3V3: now also U2.2 (VCC); no longer U2. (VCC)
- net DebugPin: now also J1.1; no longer J1.
- net GND: now also U2.1 (GND); no longer U2. (VCC)
- net SCL: now also J3.1, U2.3 (SCL); no longer J3., U2. (VCC)
- net SDA: now also J2.1, U2.4 (SDA); no longer J2., U2. (VCC)
